File: hardware/quadcopter/sensor_motion.kicad_sch (KiCad schematic)
At the start: 3 parts

Commit message: schemas and footprints
Parts:
- U?: footprint Package_LGA:LGA-14_3x2.5mm_P0.5mm_LayoutBorder3x4y -> footprints:LSM6DSO32XTR
Changed lines of the file:
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@@
     (property "Reference" "U?" (id 0) (at 91.44 46.7612 0))
     (property "Value" "LSM6DS3" (id 1) (at 91.44 49.3012 0))
-    (property "Footprint" "Package_LGA:LGA-14_3x2.5mm_P0.5mm_LayoutBorder3x4y" (id 2) (at 63.5 78.74 0)
+    (property "Footprint" "footprints:LSM6DSO32XTR" (id 2) (at 63.5 78.74 0)
       (effects (font (size 1.27 1.27)) (justify left) hide)
     )
