File: hardware/quadcopter/RF_converter.kicad_sch (KiCad schematic)
At the start: 35 parts

Commit message: schemas and footprints
Parts:
- U?: footprint Package_DFN_QFN:QFN-28-1EP_6x6mm_P0.65mm_EP4.8x4.8mm -> footprints:SX1272IMLTRT
Changed lines of the file:
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@@
       (effects (font (size 1.27 1.27)) (justify left))
     )
-    (property "Footprint" "Package_DFN_QFN:QFN-28-1EP_6x6mm_P0.65mm_EP4.8x4.8mm" (id 2) (at 85.09 93.98 0)
+    (property "Footprint" "footprints:SX1272IMLTRT" (id 2) (at 85.09 93.98 0)
       (effects (font (size 1.27 1.27)) hide)
     )

Commit message: fix
Parts:
- removed AE?: Antenna, symbol Device:Antenna
- added J?: 142-0711-821, footprints:142-0711-821, symbol 142-0711-821:142-0711-821
Connections:
- net GND: no longer C?.2, L?.2
- new net: C?.2, J?.1, L?.2
Other:
- moved on the sheet: C?
Changed lines of the file:
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@@
   (junction (at 125.73 46.99) (diameter 0) (color 0 0 0 0)
   )
-  (junction (at 252.73 66.04) (diameter 0) (color 0 0 0 0)
-  )
   (junction (at 229.87 40.64) (diameter 0) (color 0 0 0 0)
   )
@@
   (junction (at 118.11 88.9) (diameter 0) (color 0 0 0 0)
   )
+  (junction (at 248.92 66.04) (diameter 0) (color 0 0 0 0)
+  )
   (junction (at 147.32 66.04) (diameter 0) (color 0 0 0 0)
   )
@@
   )
   (junction (at 132.08 88.9) (diameter 0) (color 0 0 0 0)
-  )
-  (junction (at 265.43 66.04) (diameter 0) (color 0 0 0 0)
   )
   (junction (at 234.95 66.04) (diameter 0) (color 0 0 0 0)
@@
     (stroke (width 0) (type default) (color 0 0 0 0))
   )
-  (wire (pts (xy 266.7 67.31) (xy 265.43 67.31))
-    (stroke (width 0) (type default) (color 0 0 0 0))
-  )
   (wire (pts (xy 146.05 88.9) (xy 148.59 88.9))
     (stroke (width 0) (type default) (color 0 0 0 0))
@@
     (stroke (width 0) (type default) (color 0 0 0 0))
   )
-  (wire (pts (xy 266.7 73.66) (xy 266.7 67.31))
-    (stroke (width 0) (type default) (color 0 0 0 0))
-  )
   (wire (pts (xy 147.32 53.34) (xy 149.86 53.34))
     (stroke (width 0) (type default) (color 0 0 0 0))
@@
     (stroke (width 0) (type default) (color 0 0 0 0))
   )
-  (wire (pts (xy 265.43 67.31) (xy 265.43 66.04))
-    (stroke (width 0) (type default) (color 0 0 0 0))
-  )
   (wire (pts (xy 118.11 88.9) (xy 121.92 88.9))
     (stroke (width 0) (type default) (color 0 0 0 0))
@@
     (stroke (width 0) (type default) (color 0 0 0 0))
   )
-  (wire (pts (xy 247.65 66.04) (xy 252.73 66.04))
+  (wire (pts (xy 247.65 66.04) (xy 248.92 66.04))
     (stroke (width 0) (type default) (color 0 0 0 0))
   )
@@
     (stroke (width 0) (type default) (color 0 0 0 0))
   )
+  (wire (pts (xy 248.92 66.04) (xy 250.19 66.04))
+    (stroke (width 0) (type default) (color 0 0 0 0))
+  )
   (wire (pts (xy 226.06 40.64) (xy 229.87 40.64))
     (stroke (width 0) (type default) (color 0 0 0 0))
@@
   )
   (wire (pts (xy 219.71 60.96) (xy 219.71 92.71))
-    (stroke (width 0) (type default) (color 0 0 0 0))
-  )
-  (wire (pts (xy 252.73 66.04) (xy 265.43 66.04))
     (stroke (width 0) (type default) (color 0 0 0 0))
   )
@@
     (pin "1")
   )
+  (symbol (lib_id "142-0711-821:142-0711-821") (at 250.19 66.04 0) (unit 1)
+    (in_bom yes) (on_board yes) (fields_autoplaced)
+    (property "Reference" "J?" (id 0) (at 264.16 64.77 0)
+      (effects (font (size 1.524 1.524)) (justify left))
+    )
+    (property "Value" "142-0711-821" (id 1) (at 264.16 68.58 0)
+      (effects (font (size 1.524 1.524)) (justify left))
+    )
+    (property "Footprint" "footprints:142-0711-821" (id 2) (at 260.35 67.564 0)
+      (effects (font (size 1.524 1.524)) hide)
+    )
+    (property "Datasheet" "" (id 3) (at 250.19 66.04 0)
+      (effects (font (size 1.524 1.524)))
+    )
+    (pin "1")
+  )
   (symbol (lib_id "Device:C") (at 116.84 71.12 0) (unit 1)
     (in_bom yes) (on_board yes) (fields_autoplaced)
@@
     )
     (property "Datasheet" "" (id 3) (at 118.11 96.52 0)
-      (effects (font (size 1.27 1.27)) hide)
-    )
-    (pin "1")
-  )
-  (symbol (lib_id "power:GND") (at 266.7 73.66 0) (unit 1)
-    (in_bom yes) (on_board yes) (fields_autoplaced)
-    (property "Reference" "#PWR?" (id 0) (at 266.7 80.01 0)
-      (effects (font (size 1.27 1.27)) hide)
-    )
-    (property "Value" "GND" (id 1) (at 266.7 78.74 0))
-    (property "Footprint" "" (id 2) (at 266.7 73.66 0)
-      (effects (font (size 1.27 1.27)) hide)
-    )
-    (property "Datasheet" "" (id 3) (at 266.7 73.66 0)
       (effects (font (size 1.27 1.27)) hide)
     )
@@
     (pin "1")
     (pin "2")
-  )
-  (symbol (lib_id "Device:Antenna") (at 265.43 60.96 0) (unit 1)
-    (in_bom yes) (on_board yes) (fields_autoplaced)
-    (property "Reference" "AE?" (id 0) (at 267.97 60.3249 0)
-      (effects (font (size 1.27 1.27)) (justify left))
-    )
-    (property "Value" "Antenna" (id 1) (at 267.97 62.8649 0)
-      (effects (font (size 1.27 1.27)) (justify left))
-    )
-    (property "Footprint" "" (id 2) (at 265.43 60.96 0)
-      (effects (font (size 1.27 1.27)) hide)
-    )
-    (property "Datasheet" "~" (id 3) (at 265.43 60.96 0)
-      (effects (font (size 1.27 1.27)) hide)
-    )
-    (pin "1")
   )
   (symbol (lib_id "Device:C") (at 132.08 92.71 0) (unit 1)
@@
     (pin "2")
   )
-  (symbol (lib_id "power:GND") (at 252.73 73.66 0) (unit 1)
-    (in_bom yes) (on_board yes) (fields_autoplaced)
-    (property "Reference" "#PWR?" (id 0) (at 252.73 80.01 0)
-      (effects (font (size 1.27 1.27)) hide)
-    )
-    (property "Value" "GND" (id 1) (at 252.73 78.74 0))
-    (property "Footprint" "" (id 2) (at 252.73 73.66 0)
-      (effects (font (size 1.27 1.27)) hide)
-    )
-    (property "Datasheet" "" (id 3) (at 252.73 73.66 0)
+  (symbol (lib_id "power:GND") (at 248.92 73.66 0) (unit 1)
+    (in_bom yes) (on_board yes) (fields_autoplaced)
+    (property "Reference" "#PWR?" (id 0) (at 248.92 80.01 0)
+      (effects (font (size 1.27 1.27)) hide)
+    )
+    (property "Value" "GND" (id 1) (at 248.92 78.74 0))
+    (property "Footprint" "" (id 2) (at 248.92 73.66 0)
+      (effects (font (size 1.27 1.27)) hide)
+    )
+    (property "Datasheet" "" (id 3) (at 248.92 73.66 0)
       (effects (font (size 1.27 1.27)) hide)
     )
@@
     (pin "6")
   )
-  (symbol (lib_id "Device:C") (at 252.73 69.85 180) (unit 1)
-    (in_bom yes) (on_board yes) (fields_autoplaced)
-    (property "Reference" "C?" (id 0) (at 256.54 68.5799 0)
-      (effects (font (size 1.27 1.27)) (justify right))
-    )
-    (property "Value" "1nF" (id 1) (at 256.54 71.1199 0)
-      (effects (font (size 1.27 1.27)) (justify right))
-    )
-    (property "Footprint" "" (id 2) (at 251.7648 66.04 0)
-      (effects (font (size 1.27 1.27)) hide)
-    )
-    (property "Datasheet" "~" (id 3) (at 252.73 69.85 0)
-      (effects (font (size 1.27 1.27)) hide)
-    )
+  (symbol (lib_id "Device:C") (at 248.92 69.85 180) (unit 1)
+    (in_bom yes) (on_board yes) (fields_autoplaced)
+    (property "Reference" "C?" (id 0) (at 252.73 68.5799 0)
+      (effects (font (size 1.27 1.27)) (justify right))
+    )
+    (property "Value" "1nF" (id 1) (at 252.73 71.1199 0)
+      (effects (font (size 1.27 1.27)) (justify right))
+    )
+    (property "Footprint" "" (id 2) (at 247.9548 66.04 0)
+      (effects (font (size 1.27 1.27)) hide)
+    )
+    (property "Datasheet" "~" (id 3) (at 248.92 69.85 0)
+      (effects (font (size 1.27 1.27)) hide)
+    )

Commit message: usb req
Parts:
- removed C?: 1nF, symbol Device:C
- C?: value 1nF -> 1.834pF
- L?: value L -> 1.834nH
Changed lines of the file:
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@@
   (junction (at 118.11 88.9) (diameter 0) (color 0 0 0 0)
-  )
-  (junction (at 248.92 66.04) (diameter 0) (color 0 0 0 0)
   )
   (junction (at 147.32 66.04) (diameter 0) (color 0 0 0 0)
@@
     (stroke (width 0) (type default) (color 0 0 0 0))
   )
-  (wire (pts (xy 247.65 66.04) (xy 248.92 66.04))
+  (wire (pts (xy 247.65 66.04) (xy 250.19 66.04))
     (stroke (width 0) (type default) (color 0 0 0 0))
   )
@@
   )
   (wire (pts (xy 198.12 83.82) (xy 198.12 92.71))
-    (stroke (width 0) (type default) (color 0 0 0 0))
-  )
-  (wire (pts (xy 248.92 66.04) (xy 250.19 66.04))
     (stroke (width 0) (type default) (color 0 0 0 0))
   )
@@
     (in_bom yes) (on_board yes) (fields_autoplaced)
     (property "Reference" "L?" (id 0) (at 243.84 59.69 90))
-    (property "Value" "L" (id 1) (at 243.84 62.23 90))
+    (property "Value" "1.834nH" (id 1) (at 243.84 62.23 90))
     (property "Footprint" "" (id 2) (at 243.84 66.04 0)
       (effects (font (size 1.27 1.27)) hide)
@@
     (pin "2")
   )
-  (symbol (lib_id "power:GND") (at 248.92 73.66 0) (unit 1)
-    (in_bom yes) (on_board yes) (fields_autoplaced)
-    (property "Reference" "#PWR?" (id 0) (at 248.92 80.01 0)
-      (effects (font (size 1.27 1.27)) hide)
-    )
-    (property "Value" "GND" (id 1) (at 248.92 78.74 0))
-    (property "Footprint" "" (id 2) (at 248.92 73.66 0)
-      (effects (font (size 1.27 1.27)) hide)
-    )
-    (property "Datasheet" "" (id 3) (at 248.92 73.66 0)
-      (effects (font (size 1.27 1.27)) hide)
-    )
-    (pin "1")
-  )
   (symbol (lib_id "power:GND") (at 85.09 114.3 0) (unit 1)
     (in_bom yes) (on_board yes) (fields_autoplaced)
@@
       (effects (font (size 1.27 1.27)) (justify right))
     )
-    (property "Value" "1nF" (id 1) (at 238.76 71.1199 0)
+    (property "Value" "1.834pF" (id 1) (at 238.76 71.1199 0)
       (effects (font (size 1.27 1.27)) (justify right))
     )
@@
     (pin "6")
   )
-  (symbol (lib_id "Device:C") (at 248.92 69.85 180) (unit 1)
-    (in_bom yes) (on_board yes) (fields_autoplaced)
-    (property "Reference" "C?" (id 0) (at 252.73 68.5799 0)
-      (effects (font (size 1.27 1.27)) (justify right))
-    )
-    (property "Value" "1nF" (id 1) (at 252.73 71.1199 0)
-      (effects (font (size 1.27 1.27)) (justify right))
-    )
-    (property "Footprint" "" (id 2) (at 247.9548 66.04 0)
-      (effects (font (size 1.27 1.27)) hide)
-    )
-    (property "Datasheet" "~" (id 3) (at 248.92 69.85 0)
-      (effects (font (size 1.27 1.27)) hide)
-    )
-    (pin "1")
-    (pin "2")
-  )
 )
