File: hardware/quadcopter/power_management.kicad_sch (KiCad schematic)
At the start: 19 parts

Commit message: rf converter
Parts:
- BT1: value (none) -> Battery; footprint (none) -> Battery:BatteryHolder_Keystone_500
- CBoot? (x2), Cin? (x4), Cinx? (x2), Cout? (x2): value (none) -> C
- L? (x2): value (none) -> L
- Rfbb? (x2), Rfbt? (x2): value (none) -> R
- U? (x2): value (none) -> LMR51430XDDCR; footprint (none) -> Package_TO_SOT_SMD:SOT-23-6_Handsoldering

Commit message: usb req
Parts:
- added SUF?: SUF4001, Diode_SMD:D_MELF_Handsoldering, symbol Diode:SUF4001
Connections:
- net +5V: now also SUF?.1 (-), SUF?.2 (+)
Changed lines of the file:
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@@
   (junction (at 128.27 39.37) (diameter 0) (color 0 0 0 0)
   )
+  (junction (at 217.17 41.91) (diameter 0) (color 0 0 0 0)
+  )
   (junction (at 116.84 39.37) (diameter 0) (color 0 0 0 0)
   )
@@
     (stroke (width 0) (type default) (color 0 0 0 0))
   )
+  (wire (pts (xy 217.17 41.91) (xy 222.25 41.91))
+    (stroke (width 0) (type default) (color 0 0 0 0))
+  )
   (wire (pts (xy 170.18 128.27) (xy 161.29 128.27))
     (stroke (width 0) (type default) (color 0 0 0 0))
@@
     (stroke (width 0) (type default) (color 0 0 0 0))
   )
+  (wire (pts (xy 204.47 41.91) (xy 217.17 41.91))
+    (stroke (width 0) (type default) (color 0 0 0 0))
+  )
   (wire (pts (xy 128.27 120.65) (xy 139.7 120.65))
     (stroke (width 0) (type default) (color 0 0 0 0))
@@
     (stroke (width 0) (type default) (color 0 0 0 0))
   )
-  (wire (pts (xy 204.47 41.91) (xy 222.25 41.91))
-    (stroke (width 0) (type default) (color 0 0 0 0))
-  )
   (wire (pts (xy 172.72 41.91) (xy 185.42 41.91))
     (stroke (width 0) (type default) (color 0 0 0 0))
@@
     (stroke (width 0) (type default) (color 0 0 0 0))
   )
-  (text "Input: DC 11 V - 15 V\nOutput: 5V @ 2A" (at 194.31 27.94 0)
+  (text "Input: DC 11 V - 15 V\nOutput: 5V @ 2A" (at 184.785 24.765 0)
     (effects (font (size 1.27 1.27)) (justify left bottom))
   )
@@
     (pin "2")
   )
+  (symbol (lib_id "power:+5V") (at 217.17 29.845 0) (unit 1)
+    (in_bom yes) (on_board yes) (fields_autoplaced)
+    (property "Reference" "#PWR?" (id 0) (at 217.17 33.655 0)
+      (effects (font (size 1.27 1.27)) hide)
+    )
+    (property "Value" "+5V" (id 1) (at 217.17 24.765 0))
+    (property "Footprint" "" (id 2) (at 217.17 29.845 0)
+      (effects (font (size 1.27 1.27)) hide)
+    )
+    (property "Datasheet" "" (id 3) (at 217.17 29.845 0)
+      (effects (font (size 1.27 1.27)) hide)
+    )
+    (pin "1")
+  )
   (symbol (lib_id "power:GND") (at 158.75 67.31 0) (unit 1)
     (in_bom yes) (on_board yes) (fields_autoplaced)
@@
     (pin "1")
   )
+  (symbol (lib_id "Diode:SUF4001") (at 220.98 34.925 270) (unit 1)
+    (in_bom yes) (on_board yes) (fields_autoplaced)
+    (property "Reference" "SUF?" (id 0) (at 219.71 34.6074 90)
+      (effects (font (size 1.27 1.27)) (justify left))
+    )
+    (property "Value" "SUF4001" (id 1) (at 219.71 37.1474 90)
+      (effects (font (size 1.27 1.27)) (justify left))
+    )
+    (property "Footprint" "Diode_SMD:D_MELF_Handsoldering" (id 2) (at 219.71 34.925 0)
+      (effects (font (size 1.27 1.27)) hide)
+    )
+    (property "Datasheet" "" (id 3) (at 220.98 34.925 0)
+      (effects (font (size 1.27 1.27)) hide)
+    )
+    (pin "1")
+    (pin "2")
+  )
   (symbol (lib_id "power:GND") (at 157.48 148.59 0) (unit 1)
